File: gps_auxiliary/gps_auxiliary.brd (EAGLE design)
At the start: 61 x 59 mm, 5 parts, among them J1 FAN, J2 GPS, J3 2X6 FEMALE, U1 PYB10-Q24-S3

Commit message: Increased distance between PPS and increased power routing
Routing:
- net PPS: track 72.6 -> 70.4 mm
Other:
- board text added: "BOARD #"
Changed lines of the file:
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@@
 <vertex x="8" y="3"/>
 </polygon>
+<text x="11.5" y="2" size="1" layer="21" font="vector" ratio="12" align="center">BOARD #</text>
 </plain>
 <attributes>
@@
 <contactref element="J2" pad="1"/>
 <contactref element="J2" pad="2"/>
-<wire x1="55" y1="14" x2="55" y2="17" width="0.4" layer="1"/>
-<wire x1="56" y1="14" x2="55" y2="14" width="0.4" layer="1"/>
-<wire x1="57" y1="17" x2="57" y2="15" width="0.4" layer="1"/>
-<wire x1="57" y1="15" x2="56" y2="14" width="0.4" layer="1"/>
-<wire x1="6" y1="41" x2="2" y2="37" width="0.4" layer="1"/>
-<wire x1="2" y1="14" x2="2" y2="37" width="0.4" layer="1"/>
-<wire x1="14.16" y1="12" x2="19.16" y2="17" width="0.4" layer="1"/>
-<wire x1="4" y1="12" x2="14.16" y2="12" width="0.4" layer="1"/>
-<wire x1="4" y1="12" x2="2" y2="14" width="0.4" layer="1"/>
-<wire x1="37" y1="14" x2="34" y2="17" width="0.4" layer="1"/>
-<wire x1="34" y1="17" x2="19.16" y2="17" width="0.4" layer="1"/>
+<wire x1="55" y1="14" x2="55" y2="17" width="0.5" layer="1"/>
+<wire x1="56" y1="14" x2="55" y2="14" width="0.5" layer="1"/>
+<wire x1="57" y1="17" x2="57" y2="15" width="0.5" layer="1"/>
+<wire x1="57" y1="15" x2="56" y2="14" width="0.5" layer="1"/>
+<wire x1="6" y1="41" x2="2" y2="37" width="0.5" layer="1"/>
+<wire x1="2" y1="14" x2="2" y2="37" width="0.5" layer="1"/>
+<wire x1="14.16" y1="12" x2="19.16" y2="17" width="0.5" layer="1"/>
+<wire x1="4" y1="12" x2="14.16" y2="12" width="0.5" layer="1"/>
+<wire x1="4" y1="12" x2="2" y2="14" width="0.5" layer="1"/>
+<wire x1="37" y1="14" x2="34" y2="17" width="0.5" layer="1"/>
+<wire x1="34" y1="17" x2="19.16" y2="17" width="0.5" layer="1"/>
 <wire x1="19.16" y1="17" x2="19" y2="16.84" width="0" layer="19" extent="1-16"/>
-<wire x1="55" y1="14" x2="37" y2="14" width="0.4" layer="1"/>
+<wire x1="55" y1="14" x2="37" y2="14" width="0.5" layer="1"/>
 <wire x1="19" y1="16.84" x2="18.84" y2="16.84" width="0" layer="19" extent="1-1"/>
 </signal>
@@
 <contactref element="R1" pad="2"/>
 <contactref element="J3" pad="3"/>
-<wire x1="9.0267375" y1="25.81" x2="7.7845375" y2="27.0522" width="0.2" layer="1"/>
 <wire x1="4.73" y1="25.81" x2="5.9722" y2="27.0522" width="0.2" layer="1"/>
-<wire x1="5.9722" y1="27.0522" x2="7.7845375" y2="27.0522" width="0.2" layer="1"/>
-<wire x1="53" y1="35" x2="53" y2="31" width="0.2" layer="1"/>
-<wire x1="53" y1="31" x2="47.81" y2="25.81" width="0.2" layer="1"/>
-<wire x1="47.81" y1="25.81" x2="9.0267375" y2="25.81" width="0.2" layer="1"/>
+<wire x1="53" y1="35" x2="53" y2="33" width="0.2" layer="1"/>
+<wire x1="53" y1="33" x2="47.0522" y2="27.0522" width="0.2" layer="1"/>
+<wire x1="47.0522" y1="27.0522" x2="5.9722" y2="27.0522" width="0.2" layer="1"/>
 <wire x1="54" y1="36" x2="53" y2="35" width="0.2" layer="1"/>
 <wire x1="56" y1="36" x2="54" y2="36" width="0.2" layer="1"/>
@@
 <contactref element="J3" pad="10"/>
 <contactref element="U1" pad="2"/>
-<wire x1="7.27" y1="28.35" x2="5.62" y2="30" width="0.4" layer="1"/>
-<wire x1="5.62" y1="30" x2="4" y2="30" width="0.4" layer="1"/>
-<wire x1="4" y1="30" x2="3" y2="29" width="0.4" layer="1"/>
-<wire x1="3" y1="29" x2="3" y2="15" width="0.4" layer="1"/>
-<wire x1="3" y1="15" x2="4" y2="14" width="0.4" layer="1"/>
-<wire x1="8" y1="14" x2="9" y2="15" width="0.4" layer="1"/>
-<wire x1="9" y1="15" x2="9" y2="16.46" width="0.4" layer="1"/>
-<wire x1="9" y1="16.46" x2="7.27" y2="18.19" width="0.4" layer="1"/>
-<wire x1="4" y1="14" x2="8" y2="14" width="0.4" layer="1"/>
-<wire x1="7.27" y1="28.35" x2="20.35" y2="28.35" width="0.4" layer="1"/>
-<wire x1="26.46" y1="34.46" x2="26.46" y2="37.16" width="0.4" layer="1"/>
-<wire x1="20.35" y1="28.35" x2="26.46" y2="34.46" width="0.4" layer="1"/>
+<wire x1="7.27" y1="28.35" x2="5.62" y2="30" width="0.5" layer="1"/>
+<wire x1="5.62" y1="30" x2="4" y2="30" width="0.5" layer="1"/>
+<wire x1="4" y1="30" x2="3" y2="29" width="0.5" layer="1"/>
+<wire x1="3" y1="29" x2="3" y2="15" width="0.5" layer="1"/>
+<wire x1="3" y1="15" x2="4" y2="14" width="0.5" layer="1"/>
+<wire x1="8" y1="14" x2="9" y2="15" width="0.5" layer="1"/>
+<wire x1="9" y1="15" x2="9" y2="16.46" width="0.5" layer="1"/>
+<wire x1="9" y1="16.46" x2="7.27" y2="18.19" width="0.5" layer="1"/>
+<wire x1="4" y1="14" x2="8" y2="14" width="0.5" layer="1"/>
+<wire x1="7.27" y1="28.35" x2="20.35" y2="28.35" width="0.5" layer="1"/>
+<wire x1="26.46" y1="34.46" x2="26.46" y2="37.16" width="0.5" layer="1"/>
+<wire x1="20.35" y1="28.35" x2="26.46" y2="34.46" width="0.5" layer="1"/>
 </signal>
 </signals>
